Commit message: DELETE SECOND FLIPPER

File: src/hector_tracked_vehicles_common/hector_tracked_vehicles_description/urdf/obelix_ugv_base.urdf.xacro (robot description, xacro)
@@ -9,5 +9,5 @@
   <xacro:property name="base_link_size_z" value="0.118" />
   <xacro:property name="wheel_radius_big" value="0.085" />
-  <xacro:property name="wheel_offset_x" value="${base_link_size_x*0.5 - 0.042}" />
+  <xacro:property name="wheel_offset_x" value="${base_link_size_x*0.5}" /> <!--del -0.42-->
   <xacro:property name="wheel_offset_z" value="${base_link_size_z*0.5 - 0.065}" />
   <xacro:property name="wheel_radius"   value="0.09" />

File: src/hector_tracked_vehicles_common/hector_tracked_vehicles_description/urdf/obelix_ugv_standalone2.urdf.xacro (robot description, xacro)
@@ -9,7 +9,7 @@
     <origin xyz="${wheel_offset_x}  ${flipper_offset_y}  0 " rpy="0 0 0"/>
   </xacro:obelix_flipper_macro >
-  <xacro:obelix_flipper_macro parent="base_link" name="rear" front="-1">
+<!--  <xacro:obelix_flipper_macro parent="base_link" name="rear" front="-1">
     <origin xyz="${-wheel_offset_x}  ${flipper_offset_y}  0  " rpy="0 0 0"/>
-  </xacro:obelix_flipper_macro >
+  </xacro:obelix_flipper_macro >-->
   <gazebo reference="base_link">
     <!--<material>Gazebo/White</material>-->

Commit message: Update base link size

File: src/hector_tracked_vehicles_common/hector_tracked_vehicles_description/urdf/obelix_ugv_base.urdf.xacro (robot description, xacro)
@@ -5,13 +5,13 @@
   <!-- Properties (Constants) -->
   <xacro:property name="M_PI" value="3.14159"/>
-  <xacro:property name="base_link_size_x" value="0.52" />
-  <xacro:property name="base_link_size_y" value="0.18" />
-  <xacro:property name="base_link_size_z" value="0.118" />
-  <xacro:property name="wheel_radius_big" value="0.085" />
-  <xacro:property name="wheel_offset_x" value="${base_link_size_x*0.5}" /> <!--del -0.42-->
-  <xacro:property name="wheel_offset_z" value="${base_link_size_z*0.5 - 0.065}" />
-  <xacro:property name="wheel_radius"   value="0.09" />
-  <xacro:property name="track_width"    value="0.1" />
-  <xacro:property name="track_offset_y"    value="0.155" />
+  <xacro:property name="base_link_size_x" value="0.397" />
+  <xacro:property name="base_link_size_y" value="0.1789" /> <!--was 0.18-->
+  <xacro:property name="base_link_size_z" value="0.102" /><!-- it equal double radius, old 0.118-->
+  <xacro:property name="wheel_radius_big" value="0.1" /> <!--was 0.085--> <!--it's must be into file, but it isn't used-->
+  <xacro:property name="wheel_offset_x" value="${base_link_size_x*0.5}" /> <!--del -0.42 -->
+  <xacro:property name="wheel_offset_z" value="0" /> <!--was ${base_link_size_z*0.5-0.065}-->
+  <xacro:property name="wheel_radius"   value="0.051" /> <!--was 0.09-->
+  <xacro:property name="track_width"    value="0.04" /> <!--old 0.1-->
+  <xacro:property name="track_offset_y"    value="${base_link_size_y*0.5}" />  <!--old 0.155-->
   <xacro:property name="flipper_width"    value="0.08" />
   <xacro:property name="flipper_offset_y"    value="0.245" />
@@ -24,5 +24,5 @@
   <xacro:property name="wheel_offset_z_from_base_link" value="-0.0" />
   <xacro:property name="ground_clearance" value="0.05" />
-  <xacro:property name="top_size_x" value="0.3937" />
+  <xacro:property name="top_size_x" value="0.6" />   <!--was 0.3937-->
   <xacro:property name="top_size_y" value="0.3556" />
   <xacro:property name="top_size_z" value="0.0020" />

Commit message: Update flipper sizes in 3d model

File: src/hector_tracked_vehicles_common/hector_tracked_vehicles_description/urdf/obelix_ugv_base.urdf.xacro (robot description, xacro)
@@ -7,24 +7,24 @@
   <xacro:property name="base_link_size_x" value="0.397" />
   <xacro:property name="base_link_size_y" value="0.1789" /> <!--was 0.18-->
-  <xacro:property name="base_link_size_z" value="0.102" /><!-- it equal double radius, old 0.118-->
+  <xacro:property name="base_link_size_z" value="${2*wheel_radius-ground_clearance}" /> <!-- old 0.102 is double radius without ground_clearance 0.07683 -->
   <xacro:property name="wheel_radius_big" value="0.1" /> <!--was 0.085--> <!--it's must be into file, but it isn't used-->
   <xacro:property name="wheel_offset_x" value="${base_link_size_x*0.5}" /> <!--del -0.42 -->
-  <xacro:property name="wheel_offset_z" value="0" /> <!--was ${base_link_size_z*0.5-0.065}-->
+  <xacro:property name="wheel_offset_z" value="${-0.5*(2*wheel_radius-base_link_size_z)}" /> <!--was ${base_link_size_z*0.5-0.065 -0.012585 } -->  <!--it's difference between double radius and base-->
   <xacro:property name="wheel_radius"   value="0.051" /> <!--was 0.09-->
   <xacro:property name="track_width"    value="0.04" /> <!--old 0.1-->
   <xacro:property name="track_offset_y"    value="${base_link_size_y*0.5}" />  <!--old 0.155-->
-  <xacro:property name="flipper_width"    value="0.08" />
-  <xacro:property name="flipper_offset_y"    value="0.245" />
-  <xacro:property name="flipper_offset_wheel_axis_x"    value="0.225" />
-  <xacro:property name="wheel_length" value="0.02" />
-  <xacro:property name="wheel_size_y" value="0.0825" />
-  <xacro:property name="total_width" value="0.297" />
+  <xacro:property name="flipper_width"    value="0.028" />    <!--was 0.08-->
+  <xacro:property name="flipper_offset_y"    value="${base_link_size_y*0.5+track_width}" />  <!--old 0.245-->
+  <xacro:property name="flipper_offset_wheel_axis_x"    value="0.355" /> <!--old 0.225 -->
+  <xacro:property name="wheel_length" value="2" /> <!--i dont now how it can be used, old 0.02-->
+  <xacro:property name="wheel_size_y" value="2" /> <!--i dont now how it can be used, old 0.0825-->
+  <xacro:property name="total_width" value="2" /> <!--i dont now how it can be used, old 0.297-->
   <!--    <xacro:property name="wheel_offset_y" value="${(total_width - wheel_size_y) / 2}" />-->
-  <xacro:property name="wheel_offset_y" value="0.1697" />
-  <xacro:property name="wheel_offset_z_from_base_link" value="-0.0" />
-  <xacro:property name="ground_clearance" value="0.05" />
-  <xacro:property name="top_size_x" value="0.6" />   <!--was 0.3937-->
-  <xacro:property name="top_size_y" value="0.3556" />
-  <xacro:property name="top_size_z" value="0.0020" />
+  <xacro:property name="wheel_offset_y" value="2" /> <!--i dont now how it can be used, old 0.1697-->
+  <xacro:property name="wheel_offset_z_from_base_link" value="2" />   <!--i dont now how it can be used, old -0.0-->
+  <xacro:property name="ground_clearance" value="0" /> <!--old 0.05 0.02517-->
+  <xacro:property name="top_size_x" value="${2*(base_link_size_x+flipper_offset_wheel_axis_x)}" />  <!--was 0.3937--> <!--i dont now how it can be used-->
+  <xacro:property name="top_size_y" value="2" />  <!--was 0.3556--><!--i dont now how it can be used-->
+  <xacro:property name="top_size_z" value="2" />  <!--was 0.0020--><!--i dont now how it can be used-->
   <!--
   Note macros below are exact copies of each with expection of the

Commit message: Next stable version of packages(after Elementary reinstall)

File: src/hector_tracked_vehicles_common/hector_tracked_vehicles_description/urdf/obelix_ugv_base.urdf.xacro (robot description, xacro)
@@ -23,5 +23,5 @@
   <xacro:property name="wheel_offset_y" value="2" /> <!--i dont now how it can be used, old 0.1697-->
   <xacro:property name="wheel_offset_z_from_base_link" value="2" />   <!--i dont now how it can be used, old -0.0-->
-  <xacro:property name="ground_clearance" value="0" /> <!--old 0.05 0.02517-->
+  <xacro:property name="ground_clearance" value="0.02517" /> <!--old 0.05 0.02517-->
   <xacro:property name="top_size_x" value="${2*(base_link_size_x+flipper_offset_wheel_axis_x)}" />  <!--was 0.3937--> <!--i dont now how it can be used-->
   <xacro:property name="top_size_y" value="2" />  <!--was 0.3556--><!--i dont now how it can be used-->

Commit message: Next stable version of packages(after Elementary reinstall)

File: src/hector_tracked_vehicles_common/hector_tracked_vehicles_description/urdf/obelix_ugv_base.urdf.xacro (robot description, xacro)
@@ -23,5 +23,5 @@
   <xacro:property name="wheel_offset_y" value="2" /> <!--i dont now how it can be used, old 0.1697-->
   <xacro:property name="wheel_offset_z_from_base_link" value="2" />   <!--i dont now how it can be used, old -0.0-->
-  <xacro:property name="ground_clearance" value="0.02517" /> <!--old 0.05 0.02517-->
+  <xacro:property name="ground_clearance" value="0" /> <!--old 0.05 0.02517-->
   <xacro:property name="top_size_x" value="${2*(base_link_size_x+flipper_offset_wheel_axis_x)}" />  <!--was 0.3937--> <!--i dont now how it can be used-->
   <xacro:property name="top_size_y" value="2" />  <!--was 0.3556--><!--i dont now how it can be used-->

Commit message: Fix size of flippers

File: src/hector_tracked_vehicles_common/hector_tracked_vehicles_description/urdf/obelix_ugv_base.urdf.xacro (robot description, xacro)
@@ -13,7 +13,7 @@
   <xacro:property name="wheel_radius"   value="0.051" /> <!--was 0.09-->
   <xacro:property name="track_width"    value="0.04" /> <!--old 0.1-->
-  <xacro:property name="track_offset_y"    value="${base_link_size_y*0.5}" />  <!--old 0.155-->
+  <xacro:property name="track_offset_y"    value="${(base_link_size_y-track_width)*0.5}" />  <!--old 0.155-->
   <xacro:property name="flipper_width"    value="0.028" />    <!--was 0.08-->
-  <xacro:property name="flipper_offset_y"    value="${base_link_size_y*0.5+track_width}" />  <!--old 0.245-->
+  <xacro:property name="flipper_offset_y"    value="${0.5*(base_link_size_y+flipper_width)}" />  <!--old 0.245-->
   <xacro:property name="flipper_offset_wheel_axis_x"    value="0.355" /> <!--old 0.225 -->
   <!-- I have added it-->
