Commit message: Update URDF for track flippers

File: src/hector_tracked_vehicles_common/hector_tracked_vehicles_description/urdf/obelix_2flipper_box.urdf.xacro (robot description, xacro)
@@ -14,5 +14,5 @@
         <color rgba="0.8 0.8 0.8 1"/>
       </material>
-      <origin xyz="0 0 0" rpy="${M_PI*0.5} 0 0" />
+      <origin xyz="0 0 ${front*flipper_offset_wheel_axis_z}" rpy="${M_PI*0.5} 0 0" />
       <geometry>
         <cylinder radius="${wheel_radius}" length="${flipper_width}" />
@@ -20,19 +20,25 @@
     </visual>
     <visual>
-      <origin xyz="${front*flipper_offset_wheel_axis_x} 0 0" rpy="${M_PI*0.5} 0 0" />
+      <origin xyz="${front*flipper_offset_wheel_axis_x} 0 ${front*flipper_offset_wheel_axis_z}" rpy="${M_PI*0.5} 0 0" />
       <geometry>
-        <cylinder radius="${wheel_radius}" length="${flipper_width}" />
+        <cylinder radius="${small_flipper_wheel_radius}" length="${flipper_width}" />
       </geometry>
     </visual>
     <visual>
-      <origin xyz="${front*flipper_offset_wheel_axis_x*0.5} 0 0" rpy="0 0 0" />
+      <origin xyz="${front*flipper_offset_wheel_axis_x*0.5} 0 ${0.5*(front*flipper_offset_wheel_axis_z+wheel_radius)}" rpy="${M_PI*0.5} ${M_PI*0.5-1.4874686} 0" />
       <geometry>
-        <box size="${flipper_offset_wheel_axis_x} ${flipper_width} ${wheel_radius*2}" />
+        <box size="${flipper_offset_wheel_axis_x} ${track_thickness} ${flipper_width} " />
       </geometry>
     </visual>
-  </xacro:macro>
+    <visual>
+      <origin xyz="${front*flipper_offset_wheel_axis_x*0.5} 0 ${0.5*(2*front*flipper_offset_wheel_axis_z-wheel_radius)}" rpy="${M_PI*0.5} ${M_PI*0.5+1.4874686} 0" />
+      <geometry>
+        <box size="${flipper_offset_wheel_axis_x} ${track_thickness} ${flipper_width} " />
+      </geometry>
+    </visual>
+ </xacro:macro>
   <xacro:macro name="flipper_geom_macro_collision" params="front">
     <collision>
-      <origin xyz="0 0 0" rpy="${M_PI*0.5} 0 0" />
+      <origin xyz="0 0 ${front*flipper_offset_wheel_axis_z}" rpy="${M_PI*0.5} 0 0" />
       <geometry>
         <cylinder radius="${wheel_radius}" length="${flipper_width}" />
@@ -40,13 +46,19 @@
     </collision>
     <collision>
-      <origin xyz="${front*flipper_offset_wheel_axis_x} 0 0" rpy="${M_PI*0.5} 0 0" />
+      <origin xyz="${front*flipper_offset_wheel_axis_x} 0 ${front*flipper_offset_wheel_axis_z}" rpy="${M_PI*0.5} 0 0" />
       <geometry>
-        <cylinder radius="${wheel_radius}" length="${flipper_width}" />
+        <cylinder radius="${small_flipper_wheel_radius}" length="${flipper_width}" />
       </geometry>
     </collision>
     <collision>
-      <origin xyz="${front*flipper_offset_wheel_axis_x*0.5} 0 0" rpy="0 0 0" />
+       <origin xyz="${front*flipper_offset_wheel_axis_x*0.5} 0 ${0.5*(front*flipper_offset_wheel_axis_z+wheel_radius)}" rpy="${M_PI*0.5} ${M_PI*0.5-1.4874686} 0" />
       <geometry>
-        <box size="${flipper_offset_wheel_axis_x} ${flipper_width} ${wheel_radius*2}" />
+        <box size="${flipper_offset_wheel_axis_x} ${track_thickness} ${flipper_width} " />
+      </geometry>
+    </collision>
+   <collision>
+      <origin xyz="${front*flipper_offset_wheel_axis_x*0.5} 0 ${0.5*(2*front*flipper_offset_wheel_axis_z-wheel_radius)}" rpy="${M_PI*0.5} ${M_PI*0.5+1.4874686} 0" />
+      <geometry>
+        <box size="${flipper_offset_wheel_axis_x} ${track_thickness} ${flipper_width} " />
       </geometry>
     </collision>

File: src/hector_tracked_vehicles_common/hector_tracked_vehicles_description/urdf/obelix_ugv_base.urdf.xacro (robot description, xacro)
@@ -17,4 +17,9 @@
   <xacro:property name="flipper_offset_y"    value="${base_link_size_y*0.5+track_width}" />  <!--old 0.245-->
   <xacro:property name="flipper_offset_wheel_axis_x"    value="0.355" /> <!--old 0.225 -->
+  <!-- I have added it-->
+  <xacro:property name="flipper_offset_wheel_axis_z"    value="${wheel_offset_z}" /> <!--offset for enabled ground_clearance -->
+  <xacro:property name="small_flipper_wheel_radius"    value="0.02135" /> <!--offset for enabled ground_clearance old 0.0427/2-->
+  <xacro:property name="track_thickness"    value="0.005" /> <!--offset for enabled ground_clearance old 0.0427/2-->
+  <!---->
   <xacro:property name="wheel_length" value="2" /> <!--i dont now how it can be used, old 0.02-->
   <xacro:property name="wheel_size_y" value="2" /> <!--i dont now how it can be used, old 0.0825-->
@@ -23,5 +28,5 @@
   <xacro:property name="wheel_offset_y" value="2" /> <!--i dont now how it can be used, old 0.1697-->
   <xacro:property name="wheel_offset_z_from_base_link" value="2" />   <!--i dont now how it can be used, old -0.0-->
-  <xacro:property name="ground_clearance" value="0" /> <!--old 0.05 0.02517-->
+  <xacro:property name="ground_clearance" value="0.02517" /> <!--old 0.05 0.02517-->
   <xacro:property name="top_size_x" value="${2*(base_link_size_x+flipper_offset_wheel_axis_x)}" />  <!--was 0.3937--> <!--i dont now how it can be used-->
   <xacro:property name="top_size_y" value="2" />  <!--was 0.3556--><!--i dont now how it can be used-->

Commit message: Robot model not crash in Gazebo

File: src/hector_tracked_vehicles_common/hector_tracked_vehicles_description/urdf/obelix_2flipper_box.urdf.xacro (robot description, xacro)
@@ -1,4 +1,5 @@
 <?xml version="1.0"?>
 <robot xmlns:xacro="http://www.ros.org/wiki/xacro">
+  <!--xacro:include filename="$(find hector_tracked_vehicles_description)/urdf/tracked_wheel.urdf.xacro" /-->
   <xacro:property name="flipper_base_mass" value="2.0"/>
   <xacro:property name="flipper_x" value="0.3"/>
@@ -32,5 +33,5 @@
     </visual>
     <visual>
-      <origin xyz="${front*flipper_offset_wheel_axis_x*0.5} 0 ${0.5*(2*front*flipper_offset_wheel_axis_z-wheel_radius)}" rpy="${M_PI*0.5} ${M_PI*0.5+1.4874686} 0" />
+      <origin xyz="${front*flipper_offset_wheel_axis_x*0.5} 0 ${0.5*(front*flipper_offset_wheel_axis_z-wheel_radius)}" rpy="${M_PI*0.5} ${M_PI*0.5+1.4874686} 0" />
       <geometry>
         <box size="${flipper_offset_wheel_axis_x} ${track_thickness} ${flipper_width} " />
@@ -58,5 +59,5 @@
     </collision>
    <collision>
-      <origin xyz="${front*flipper_offset_wheel_axis_x*0.5} 0 ${0.5*(2*front*flipper_offset_wheel_axis_z-wheel_radius)}" rpy="${M_PI*0.5} ${M_PI*0.5+1.4874686} 0" />
+      <origin xyz="${front*flipper_offset_wheel_axis_x*0.5} 0 ${0.5*(front*flipper_offset_wheel_axis_z-wheel_radius)}" rpy="${M_PI*0.5} ${M_PI*0.5+1.4874686} 0" />
       <geometry>
         <box size="${flipper_offset_wheel_axis_x} ${track_thickness} ${flipper_width} " />

File: src/hector_tracked_vehicles_common/hector_tracked_vehicles_description/urdf/obelix_ugv_base.urdf.xacro (robot description, xacro)
@@ -13,7 +13,7 @@
   <xacro:property name="wheel_radius"   value="0.051" /> <!--was 0.09-->
   <xacro:property name="track_width"    value="0.04" /> <!--old 0.1-->
-  <xacro:property name="track_offset_y"    value="${(base_link_size_y-track_width)*0.5}" />  <!--old 0.155-->
+  <xacro:property name="track_offset_y"    value="${(base_link_size_y-flipper_width)*0.5}" />  <!--old 0.155-->
   <xacro:property name="flipper_width"    value="0.028" />    <!--was 0.08-->
-  <xacro:property name="flipper_offset_y"    value="${0.5*(base_link_size_y+flipper_width)}" />  <!--old 0.245-->
+  <xacro:property name="flipper_offset_y"    value="${0.5*(base_link_size_y+*track_width)}" />  <!--old 0.245-->
   <xacro:property name="flipper_offset_wheel_axis_x"    value="0.355" /> <!--old 0.225 -->
   <!-- I have added it-->

File: src/hector_tracked_vehicles_common/hector_tracked_vehicles_description/urdf/obelix_ugv_standalone2.urdf.xacro (robot description, xacro)
@@ -9,7 +9,7 @@
     <origin xyz="${wheel_offset_x}  ${flipper_offset_y}  0 " rpy="0 0 0"/>
   </xacro:obelix_flipper_macro >
-<!--  <xacro:obelix_flipper_macro parent="base_link" name="rear" front="-1">
-    <origin xyz="${-wheel_offset_x}  ${flipper_offset_y}  0  " rpy="0 0 0"/>
-  </xacro:obelix_flipper_macro >-->
+  <xacro:obelix_flipper_macro parent="base_link" name="rear" front="1">
+    <origin xyz="${-wheel_offset_x+base_link_size_x}  ${flipper_offset_y}  0  " rpy="0 0 0"/>
+  </xacro:obelix_flipper_macro >
   <gazebo reference="base_link">
     <!--<material>Gazebo/White</material>-->
