Commit message: Kill inertia

File: src/gazebo_ros_demos/rrbot_description/urdf/rrbot.xacro (robot description, xacro)
@@ -5,8 +5,8 @@
   <xacro:property name="PI" value="3.1415926535897931"/>
   <xacro:property name="mass" value="1" /> <!-- arbitrary value for mass -->
-  <xacro:property name="width" value="0.1" /> <!-- Square dimensions (widthxwidth) of beams -->
-  <xacro:property name="height1" value="2" /> <!-- Link 1 -->
-  <xacro:property name="height2" value="1" /> <!-- Link 2 -->
-  <xacro:property name="height3" value="1" /> <!-- Link 3 -->
+  <xacro:property name="width" value="0" /> <!-- Square dimensions (widthxwidth) of beams  0.1-->
+  <xacro:property name="height1" value="0" /> <!-- Link 1 2  -->
+  <xacro:property name="height2" value="0" /> <!-- Link 2 1  -->
+  <xacro:property name="height3" value="0" /> <!-- Link 3 1 -->
   <xacro:property name="camera_link" value="0.05" /> <!-- Size of square 'camera' box -->
   <xacro:property name="axel_offset" value="0.05" /> <!-- Space btw top of beam and the each joint -->

Commit message: Testing. Start working on Today

File: src/gazebo_ros_demos/rrbot_description/urdf/rrbot.xacro (robot description, xacro)
@@ -3,5 +3,5 @@
 <robot name="rrbot" xmlns:xacro="http://www.ros.org/wiki/xacro">
   <!-- Constants for robot dimensions -->
-  <xacro:property name="PI" value="3.1415926535897931"/>
+  <xacro:property name="PI" value="3.1415"/>
   <xacro:property name="mass" value="1" /> <!-- arbitrary value for mass -->
   <xacro:property name="width" value="0" /> <!-- Square dimensions (widthxwidth) of beams  0.1-->
@@ -21,45 +21,40 @@
   <xacro:include filename="$(find rrbot_description)/urdf/materials.xacro" />
   <!-- Used for fixing robot to Gazebo 'base_link' -->
-  <link name="world"/>
-  <joint name="fixed" type="fixed">
-    <parent link="world"/>
-    <child link="link1"/>
-  </joint>
   <!-- Base Link -->
   <link name="link1">
     <collision>
-      <origin xyz="0 0 ${base_link_size_z/2}" rpy="${PI*0.5} 0 ${PI*0.5} "/>
+      <origin xyz="0 0 0" rpy="0 0 0"/>
       <geometry>
-        <!--box size="${width} ${width} ${height1}"/-->
-        <mesh filename="package://rrbot_description/meshes/base_link.stl"/>
+        <mesh filename="package://rrbot_description/meshes/base_link_3.stl"/>
       </geometry>
     </collision>
     <visual>
-      <origin xyz="0 0 ${base_link_size_z/2}" rpy="${PI*0.5} 0 ${PI*0.5} "/>
+      <origin xyz="0 0 0" rpy="0 0 0"/>
       <geometry>
-        <mesh filename="package://rrbot_description/meshes/base_link.stl"/>
+        <mesh filename="package://rrbot_description/meshes/base_link_3.stl"/>
       </geometry>
       <material name="orange"/>
     </visual>
     <inertial>
-      <origin xyz="0 0 ${base_link_size_z/2}" rpy="${PI*0.5} 0 ${PI*0.5}"/>
+      <origin xyz="0 0 0" rpy="0 0 0"/>
       <mass value="${mass}"/>
       <inertia
-	  ixx="${mass / 12.0 * (width*width + height1*height1)}" ixy="0.0" ixz="0.0"
-	  iyy="${mass / 12.0 * (height1*height1 + width*width)}" iyz="0.0"
-	  izz="${mass / 12.0 * (width*width + width*width)}"/>
+	  ixx="1" ixy="0.0" ixz="0.0"
+	  iyy="1" iyz="0.0"
+	  izz="1"/>
     </inertial>
   </link>
-  <joint name="joint1" type="continuous">
+  <joint name="joint1" type="revolute">
     <parent link="link1"/>
     <child link="link2"/>
     <origin xyz="${base_link_size_x*0.0} 0 ${base_link_size_z*0.5}" rpy="0 0 0"/>
     <axis xyz="0 1 0"/>
-    <dynamics damping="0.7"/>
+    <!--dynamics damping="0.7"/-->
+    <limit lower="${-PI*0.5}" upper="${PI*0.5}" effort="100" velocity="1"/>
   </joint>
   <!-- Middle Link -->
   <link name="link2">
     <collision>
-      <origin xyz="0 0 0" rpy="${PI*0.5} 0 ${PI*0.5}"/>
+      <origin xyz="0 0 0" rpy="0 0 0"/>
       <geometry>
         <mesh filename="package://rrbot_description/meshes/left_flipper.stl"/>
@@ -67,5 +62,5 @@
     </collision>
     <visual>
-      <origin xyz="0 0 0" rpy="${PI*0.5} 0 ${PI*0.5}"/>
+      <origin xyz="0 0 0" rpy="0 0 0"/>
       <geometry>
         <mesh filename="package://rrbot_description/meshes/left_flipper.stl"/>
@@ -74,13 +69,13 @@
     </visual>
     <inertial>
-      <origin xyz="0 0 0" rpy="${PI*0.5} 0 ${PI*0.5}"/>
+      <origin xyz="0 0 0" rpy="0 0 0"/>
       <mass value="${mass}"/>
       <inertia
-	  ixx="${mass / 12.0 * (width*width + height2*height2)}" ixy="0.0" ixz="0.0"
-	  iyy="${mass / 12.0 * (height2*height2 + width*width)}" iyz="0.0"
-	  izz="${mass / 12.0 * (width*width + width*width)}"/>
+	  ixx="1" ixy="0.0" ixz="0.0"
+	  iyy="1" iyz="0.0"
+	  izz="1"/>
     </inertial>
   </link>
-  <joint name="joint2" type="continuous">
+  <!--joint name="joint2" type="revolute">
     <parent link="link1"/>
     <child link="link3"/>
@@ -88,9 +83,10 @@
     <axis xyz="0 1 0"/>
     <dynamics damping="0.7"/>
-  </joint>
+    <limit lower="${-PI*0.5}" upper="${PI*0.5}" effort="100" velocity="1"/>
+  </joint-->
   <!-- Top Link -->
-  <link name="link3">
+  <!--link name="link3">
     <collision>
-      <origin xyz="0 0 0" rpy="${-PI*0.5} 0 ${-PI*0.5}"/>
+      <origin xyz="0 0 0" rpy="0 0 0"/>
       <geometry>
         <mesh filename="package://rrbot_description/meshes/right_flipper.stl"/>
@@ -98,5 +94,5 @@
     </collision>
     <visual>
-      <origin xyz="0 0 0" rpy="${-PI*0.5} 0 ${-PI*0.5}"/>
+      <origin xyz="0 0 0" rpy="0 0 0"/>
       <geometry>
         <mesh filename="package://rrbot_description/meshes/right_flipper.stl"/>
@@ -105,20 +101,20 @@
     </visual>
     <inertial>
-      <origin xyz="0 0 0" rpy="${-PI*0.5} 0 ${-PI*0.5}"/>
+      <origin xyz="0 0 0" rpy="0 0 0"/>
       <mass value="${mass}"/>
       <inertia
-	  ixx="${mass / 12.0 * (width*width + height3*height3)}" ixy="0.0" ixz="0.0"
-	  iyy="${mass / 12.0 * (height3*height3 + width*width)}" iyz="0.0"
-	  izz="${mass / 12.0 * (width*width + width*width)}"/>
+	  ixx="1" ixy="0.0" ixz="0.0"
+	  iyy="1" iyz="0.0"
+	  izz="1"/>
     </inertial>
-  </link>
-  <joint name="hokuyo_joint" type="fixed">
+  </link-->
+  <!--joint name="hokuyo_joint" type="fixed">
     <axis xyz="0 1 0" />
     <origin xyz="0 0 ${height3 - axel_offset/2}" rpy="0 0 0"/>
     <parent link="world"/>
     <child link="hokuyo_link"/>
-  </joint>
+  </joint-->
   <!-- Hokuyo Laser -->
-  <link name="hokuyo_link">
+  <!--link name="hokuyo_link">
     <collision>
       <origin xyz="0 0 0" rpy="0 0 0"/>
@@ -138,13 +134,13 @@
       <inertia ixx="1e-6" ixy="0" ixz="0" iyy="1e-6" iyz="0" izz="1e-6" />
     </inertial>
-  </link>
-  <joint name="camera_joint" type="fixed">
+  </link-->
+  <!--joint name="camera_joint" type="fixed">
     <axis xyz="0 1 0" />
     <origin xyz="${camera_link} 0 ${height3 - axel_offset*2}" rpy="0 0 0"/>
     <parent link="world"/>
     <child link="camera_link"/>
-  </joint>
+  </joint-->
   <!-- Camera -->
-  <link name="camera_link">
+  <!--link name="camera_link">
     <collision>
       <origin xyz="0 0 0" rpy="0 0 0"/>
@@ -165,6 +161,6 @@
       <inertia ixx="1e-6" ixy="0" ixz="0" iyy="1e-6" iyz="0" izz="1e-6" />
     </inertial>
-  </link>
-  <transmission name="tran1">
+  </link-->
+  <!--transmission name="tran1">
     <type>transmission_interface/SimpleTransmission</type>
     <joint name="joint1">
@@ -175,12 +171,12 @@
       <mechanicalReduction>1</mechanicalReduction>
     </actuator>
-  </transmission>
+  </transmission-->
   <transmission name="tran2">
     <type>transmission_interface/SimpleTransmission</type>
     <joint name="joint2">
-      <hardwareInterface>EffortJointInterface</hardwareInterface>
+      <hardwareInterface>PositionJointInterface</hardwareInterface>
     </joint>
     <actuator name="motor2">
-      <hardwareInterface>EffortJointInterface</hardwareInterface>
+      <hardwareInterface>PositionJointInterface</hardwareInterface>
       <mechanicalReduction>1</mechanicalReduction>
     </actuator>

Commit message: Create good-managed mesh model

File: src/gazebo_ros_demos/rrbot_description/urdf/rrbot.xacro (robot description, xacro)
@@ -11,6 +11,6 @@
   <xacro:property name="camera_link" value="0.05" /> <!-- Size of square 'camera' box -->
   <xacro:property name="axel_offset" value="0.05" /> <!-- Space btw top of beam and the each joint -->
-  <xacro:property name="base_link_size_x" value="0.397" />
-  <xacro:property name="base_link_size_y" value="0.1789" /> <!--was 0.18-->
+  <xacro:property name="base_link_size_x" value="0.1789" /> <!--was 0.397-->
+  <xacro:property name="base_link_size_y" value="0.397" /> <!--was 0.1789-->
   <xacro:property name="base_link_size_z" value="${2*wheel_radius-ground_clearance}" /> <!-- old 0.102 is double radius without ground_clearance 0.07683 -->
   <xacro:property name="wheel_radius"   value="0.051" /> <!--was 0.09-->
@@ -20,23 +20,21 @@
   <!-- Import Rviz colors -->
   <xacro:include filename="$(find rrbot_description)/urdf/materials.xacro" />
-  <!-- Used for fixing robot to Gazebo 'base_link' -->
-  <!-- Base Link -->
   <link name="link1">
+    <visual>
+      <origin xyz="0 0 0" rpy="0 0 0 "/>
+      <geometry>
+        <mesh filename="package://rrbot_description/meshes/base_link2.dae"/>
+      </geometry>
+      <material name="orange"/>
+    </visual>
     <collision>
       <origin xyz="0 0 0" rpy="0 0 0"/>
       <geometry>
-        <mesh filename="package://rrbot_description/meshes/base_link_3.stl"/>
+        <mesh filename="package://rrbot_description/meshes/base_link2.dae"/>
       </geometry>
     </collision>
-    <visual>
-      <origin xyz="0 0 0" rpy="0 0 0"/>
-      <geometry>
-        <mesh filename="package://rrbot_description/meshes/base_link_3.stl"/>
-      </geometry>
-      <material name="orange"/>
-    </visual>
     <inertial>
-      <origin xyz="0 0 0" rpy="0 0 0"/>
-      <mass value="${mass}"/>
+      <origin xyz="0 ${-base_link_size_y*0.5} 0" rpy="0 0 0 "/>
+      <mass value="${1000*mass}"/>
       <inertia
 	  ixx="1" ixy="0.0" ixz="0.0"
@@ -48,15 +46,13 @@
     <parent link="link1"/>
     <child link="link2"/>
-    <origin xyz="${base_link_size_x*0.0} 0 ${base_link_size_z*0.5}" rpy="0 0 0"/>
-    <axis xyz="0 1 0"/>
-    <!--dynamics damping="0.7"/-->
-    <limit lower="${-PI*0.5}" upper="${PI*0.5}" effort="100" velocity="1"/>
+    <origin xyz="0 0 0 " rpy="${PI*0.0} ${PI*0.0} ${PI*0.0}"/>
+    <axis xyz="1 0 0"/>
+    <limit lower="${-PI*0.0}" upper="${PI*0.5}" effort="100" velocity="1"/>
   </joint>
-  <!-- Middle Link -->
   <link name="link2">
     <collision>
       <origin xyz="0 0 0" rpy="0 0 0"/>
       <geometry>
-        <mesh filename="package://rrbot_description/meshes/left_flipper.stl"/>
+        <mesh filename="package://rrbot_description/meshes/left_flipper2.dae"/>
       </geometry>
     </collision>
@@ -64,11 +60,11 @@
       <origin xyz="0 0 0" rpy="0 0 0"/>
       <geometry>
-        <mesh filename="package://rrbot_description/meshes/left_flipper.stl"/>
+        <mesh filename="package://rrbot_description/meshes/left_flipper2.dae"/>
       </geometry>
-      <material name="blue"/>
+      <material name="grey"/>
     </visual>
     <inertial>
       <origin xyz="0 0 0" rpy="0 0 0"/>
-      <mass value="${mass}"/>
+      <mass value="${0.0001*mass}"/>
       <inertia
 	  ixx="1" ixy="0.0" ixz="0.0"
@@ -77,18 +73,16 @@
     </inertial>
   </link>
-  <!--joint name="joint2" type="revolute">
+  <joint name="joint2" type="revolute">
     <parent link="link1"/>
     <child link="link3"/>
-    <origin xyz="0 0 ${base_link_size_z*0.5}" rpy="0 0 0"/>
-    <axis xyz="0 1 0"/>
-    <dynamics damping="0.7"/>
-    <limit lower="${-PI*0.5}" upper="${PI*0.5}" effort="100" velocity="1"/>
-  </joint-->
-  <!-- Top Link -->
-  <!--link name="link3">
+    <origin xyz="0 0 0" rpy="0 0 0"/>
+    <axis xyz="1 0 0"/>
+    <limit lower="${-PI*0.0}" upper="${PI*0.5}" effort="100" velocity="1"/>
+  </joint>
+  <link name="link3">
     <collision>
       <origin xyz="0 0 0" rpy="0 0 0"/>
       <geometry>
-        <mesh filename="package://rrbot_description/meshes/right_flipper.stl"/>
+        <mesh filename="package://rrbot_description/meshes/right_flipper2.dae"/>
       </geometry>
     </collision>
@@ -96,11 +90,11 @@
       <origin xyz="0 0 0" rpy="0 0 0"/>
       <geometry>
-        <mesh filename="package://rrbot_description/meshes/right_flipper.stl"/>
+        <mesh filename="package://rrbot_description/meshes/right_flipper2.dae"/>
       </geometry>
-      <material name="blue"/>
+      <material name="grey"/>
     </visual>
     <inertial>
       <origin xyz="0 0 0" rpy="0 0 0"/>
-      <mass value="${mass}"/>
+      <mass value="${0.0001*mass}"/>
       <inertia
 	  ixx="1" ixy="0.0" ixz="0.0"
@@ -108,5 +102,5 @@
 	  izz="1"/>
     </inertial>
-  </link-->
+  </link>
   <!--joint name="hokuyo_joint" type="fixed">
     <axis xyz="0 1 0" />
@@ -162,5 +156,5 @@
     </inertial>
   </link-->
-  <!--transmission name="tran1">
+  <transmission name="tran1">
     <type>transmission_interface/SimpleTransmission</type>
     <joint name="joint1">
@@ -171,12 +165,12 @@
       <mechanicalReduction>1</mechanicalReduction>
     </actuator>
-  </transmission-->
+  </transmission>
   <transmission name="tran2">
     <type>transmission_interface/SimpleTransmission</type>
     <joint name="joint2">
-      <hardwareInterface>PositionJointInterface</hardwareInterface>
+      <hardwareInterface>EffortJointInterface</hardwareInterface>
     </joint>
     <actuator name="motor2">
-      <hardwareInterface>PositionJointInterface</hardwareInterface>
+      <hardwareInterface>>EffortJointInterface</hardwareInterface>
       <mechanicalReduction>1</mechanicalReduction>
     </actuator>

Commit message: Add rrbot_control to rrbot_gazebo running

File: src/gazebo_ros_demos/rrbot_description/urdf/rrbot.xacro (robot description, xacro)
@@ -36,5 +36,5 @@
     <inertial>
       <origin xyz="0 ${-base_link_size_y*0.5} 0" rpy="0 0 0 "/>
-      <mass value="${1000*mass}"/>
+      <mass value="${5*mass}"/>
       <inertia
 	  ixx="1" ixy="0.0" ixz="0.0"
@@ -48,5 +48,5 @@
     <origin xyz="0 0 0 " rpy="${PI*0.0} ${PI*0.0} ${PI*0.0}"/>
     <axis xyz="1 0 0"/>
-    <limit lower="${-PI*0.0}" upper="${PI*0.5}" effort="100" velocity="1"/>
+    <limit lower="${-PI*0.5}" upper="${PI*0.5}" effort="100" velocity="1"/>
   </joint>
   <link name="link2">
@@ -66,5 +66,5 @@
     <inertial>
       <origin xyz="0 0 0" rpy="0 0 0"/>
-      <mass value="${0.0001*mass}"/>
+      <mass value="${1*mass}"/>
       <inertia
 	  ixx="1" ixy="0.0" ixz="0.0"
@@ -78,5 +78,5 @@
     <origin xyz="0 0 0" rpy="0 0 0"/>
     <axis xyz="1 0 0"/>
-    <limit lower="${-PI*0.0}" upper="${PI*0.5}" effort="100" velocity="1"/>
+    <limit lower="${-PI*0.5}" upper="${PI*0.5}" effort="100" velocity="1"/>
   </joint>
   <link name="link3">
@@ -96,5 +96,5 @@
     <inertial>
       <origin xyz="0 0 0" rpy="0 0 0"/>
-      <mass value="${0.0001*mass}"/>
+      <mass value="${1*mass}"/>
       <inertia
 	  ixx="1" ixy="0.0" ixz="0.0"
