Commit message: Add synchronization and movement forward

File: src/gazebo_ros_demos/rrbot_description/urdf/rrbot.xacro (robot description, xacro)
@@ -1,19 +1,31 @@
-<?xml version="1.0"?>
+<?xml version="1.0" encoding="UTF-8"?>
 <!-- Revolute-Revolute Manipulator -->
 <robot name="rrbot" xmlns:xacro="http://www.ros.org/wiki/xacro">
   <!-- Constants for robot dimensions -->
   <xacro:property name="PI" value="3.1415"/>
-  <xacro:property name="mass" value="1" /> <!-- arbitrary value for mass -->
-  <xacro:property name="width" value="0" /> <!-- Square dimensions (widthxwidth) of beams  0.1-->
-  <xacro:property name="height1" value="0" /> <!-- Link 1 2  -->
-  <xacro:property name="height2" value="0" /> <!-- Link 2 1  -->
-  <xacro:property name="height3" value="0" /> <!-- Link 3 1 -->
-  <xacro:property name="camera_link" value="0.05" /> <!-- Size of square 'camera' box -->
-  <xacro:property name="axel_offset" value="0.05" /> <!-- Space btw top of beam and the each joint -->
-  <xacro:property name="base_link_size_x" value="0.1789" /> <!--was 0.397-->
-  <xacro:property name="base_link_size_y" value="0.397" /> <!--was 0.1789-->
-  <xacro:property name="base_link_size_z" value="${2*wheel_radius-ground_clearance}" /> <!-- old 0.102 is double radius without ground_clearance 0.07683 -->
-  <xacro:property name="wheel_radius"   value="0.051" /> <!--was 0.09-->
-    <xacro:property name="ground_clearance" value="0.02517" /> <!--old 0.05 0.02517-->
+  <xacro:property name="mass" value="1" />
+  <!-- arbitrary value for mass -->
+  <xacro:property name="width" value="0" />
+  <!-- Square dimensions (widthxwidth) of beams  0.1-->
+  <xacro:property name="height1" value="0" />
+  <!-- Link 1 2  -->
+  <xacro:property name="height2" value="0" />
+  <!-- Link 2 1  -->
+  <xacro:property name="height3" value="0" />
+  <!-- Link 3 1 -->
+  <xacro:property name="camera_link" value="0.05" />
+  <!-- Size of square 'camera' box -->
+  <xacro:property name="axel_offset" value="0.05" />
+  <!-- Space btw top of beam and the each joint -->
+  <xacro:property name="base_link_size_x" value="0.1789" />
+  <!--was 0.397-->
+  <xacro:property name="base_link_size_y" value="0.397" />
+  <!--was 0.1789-->
+  <xacro:property name="base_link_size_z" value="${2*wheel_radius-ground_clearance}" />
+  <!-- old 0.102 is double radius without ground_clearance 0.07683 -->
+  <xacro:property name="wheel_radius"   value="0.051" />
+  <!--was 0.09-->
+  <xacro:property name="ground_clearance" value="0.02517" />
+  <!--old 0.05 0.02517-->
   <!-- Import all Gazebo-customization elements, including Gazebo colors -->
   <xacro:include filename="$(find rrbot_description)/urdf/rrbot.gazebo" />
@@ -37,8 +49,5 @@
       <origin xyz="0 ${-base_link_size_y*0.5} 0" rpy="0 0 0 "/>
       <mass value="${5*mass}"/>
-      <inertia
-	  ixx="1" ixy="0.0" ixz="0.0"
-	  iyy="1" iyz="0.0"
-	  izz="1"/>
+      <inertia	  ixx="1" ixy="0.0" ixz="0.0"	  iyy="1" iyz="0.0"	  izz="1"/>
     </inertial>
   </link>
@@ -67,8 +76,5 @@
       <origin xyz="0 0 0" rpy="0 0 0"/>
       <mass value="${1*mass}"/>
-      <inertia
-	  ixx="1" ixy="0.0" ixz="0.0"
-	  iyy="1" iyz="0.0"
-	  izz="1"/>
+      <inertia	  ixx="1" ixy="0.0" ixz="0.0"	  iyy="1" iyz="0.0"	  izz="1"/>
     </inertial>
   </link>
@@ -97,82 +103,152 @@
       <origin xyz="0 0 0" rpy="0 0 0"/>
       <mass value="${1*mass}"/>
-      <inertia
-	  ixx="1" ixy="0.0" ixz="0.0"
-	  iyy="1" iyz="0.0"
-	  izz="1"/>
-    </inertial>
-  </link>
+      <inertia	  ixx="1" ixy="0.0" ixz="0.0"	  iyy="1" iyz="0.0"	  izz="1"/>
+    </inertial>
+  </link>
+  <link name="link4">
+    <collision>
+      <origin xyz="0.00 0 0.0" rpy="0 ${PI*0.5} 0"/>
+      <geometry>
+        <cylinder radius='${wheel_radius*1.4}' length="0.02"/>
+      </geometry>
+    </collision>
+    <visual>
+      <origin xyz="0.00 0 0.00" rpy="0 ${PI*0.5} 0"/>
+      <geometry>
+        <cylinder radius='${wheel_radius*1.4}' length="0.02"/>
+      </geometry>
+      <material name="red"/>
+    </visual>
+    <inertial>
+      <origin xyz="0.00 0 0.00" rpy="0 ${PI*0.5} 0"/>
+      <mass value="${0.001*mass}"/>
+      <inertia	  ixx="1" ixy="0.0" ixz="0.0"	  iyy="1" iyz="0.0"	  izz="1"/>
+    </inertial>
+  </link>
+  <joint name="joint3" type="continuous">
+    <parent link="link2"/>
+    <child link="link4"/>
+    <origin xyz="${base_link_size_x*3/2} 0 0 " rpy="${PI*0.0} ${PI*0.0} ${PI*0.0}"/>
+    <axis xyz="1 0 0"/>
+    <!--limit lower="${-PI}" upper="${PI}" effort="100" velocity="1"/-->
+  </joint>
+  <link name="link5">
+    <collision>
+      <origin xyz="0.00 0 0.0" rpy="0 ${PI*0.5} 0"/>
+      <geometry>
+        <cylinder radius='${wheel_radius*1.4}' length="0.02"/>
+      </geometry>
+    </collision>
+    <visual>
+      <origin xyz="0.00 0 0.00" rpy="0 ${PI*0.5} 0"/>
+      <geometry>
+        <cylinder radius='${wheel_radius*1.4}' length="0.02"/>
+      </geometry>
+      <material name="red"/>
+    </visual>
+    <inertial>
+      <origin xyz="0.00 0 0.00" rpy="0 ${PI*0.5} 0"/>
+      <mass value="${0.001*mass}"/>
+      <inertia	  ixx="1" ixy="0.0" ixz="0.0"	  iyy="1" iyz="0.0"	  izz="1"/>
+    </inertial>
+  </link>
+  <joint name="joint4" type="continuous">
+    <parent link="link3"/>
+    <child link="link5"/>
+    <origin xyz="${-base_link_size_x*3/2} 0 0 " rpy="${PI*0.0} ${PI*0.0} ${PI*0.0}"/>
+    <axis xyz="1 0 0"/>
+  </joint>
   <!--joint name="hokuyo_joint" type="fixed">
-    <axis xyz="0 1 0" />
-    <origin xyz="0 0 ${height3 - axel_offset/2}" rpy="0 0 0"/>
-    <parent link="world"/>
-    <child link="hokuyo_link"/>
-  </joint-->
-  <!-- Hokuyo Laser -->
-  <!--link name="hokuyo_link">
-    <collision>
-      <origin xyz="0 0 0" rpy="0 0 0"/>
-      <geometry>
-	<box size="0.1 0.1 0.1"/>
-      </geometry>
-    </collision>
-    <visual>
-      <origin xyz="0 0 0" rpy="0 0 0"/>
-      <geometry>
-        <mesh filename="package://rrbot_description/meshes/hokuyo.dae"/>
-      </geometry>
-    </visual>
-    <inertial>
-      <mass value="1e-5" />
-      <origin xyz="0 0 0" rpy="0 0 0"/>
-      <inertia ixx="1e-6" ixy="0" ixz="0" iyy="1e-6" iyz="0" izz="1e-6" />
-    </inertial>
-  </link-->
-  <!--joint name="camera_joint" type="fixed">
-    <axis xyz="0 1 0" />
-    <origin xyz="${camera_link} 0 ${height3 - axel_offset*2}" rpy="0 0 0"/>
-    <parent link="world"/>
-    <child link="camera_link"/>
-  </joint-->
-  <!-- Camera -->
-  <!--link name="camera_link">
-    <collision>
-      <origin xyz="0 0 0" rpy="0 0 0"/>
-      <geometry>
-	<box size="${camera_link} ${camera_link} ${camera_link}"/>
-      </geometry>
-    </collision>
-    <visual>
-      <origin xyz="0 0 0" rpy="0 0 0"/>
-      <geometry>
-	<box size="${camera_link} ${camera_link} ${camera_link}"/>
-      </geometry>
-      <material name="red"/>
-    </visual>
-    <inertial>
-      <mass value="1e-5" />
-      <origin xyz="0 0 0" rpy="0 0 0"/>
-      <inertia ixx="1e-6" ixy="0" ixz="0" iyy="1e-6" iyz="0" izz="1e-6" />
-    </inertial>
-  </link-->
-  <transmission name="tran1">
-    <type>transmission_interface/SimpleTransmission</type>
-    <joint name="joint1">
-      <hardwareInterface>EffortJointInterface</hardwareInterface>
-    </joint>
-    <actuator name="motor1">
-      <hardwareInterface>EffortJointInterface</hardwareInterface>
-      <mechanicalReduction>1</mechanicalReduction>
-    </actuator>
-  </transmission>
-  <transmission name="tran2">
-    <type>transmission_interface/SimpleTransmission</type>
-    <joint name="joint2">
-      <hardwareInterface>EffortJointInterface</hardwareInterface>
-    </joint>
-    <actuator name="motor2">
-      <hardwareInterface>>EffortJointInterface</hardwareInterface>
-      <mechanicalReduction>1</mechanicalReduction>
-    </actuator>
-  </transmission>
+  <axis xyz="0 1 0" />
+  <origin xyz="0 0 ${height3 - axel_offset/2}" rpy="0 0 0"/>
+  <parent link="world"/>
+  <child link="hokuyo_link"/>
+</joint-->
+<!-- Hokuyo Laser -->
+<!--link name="hokuyo_link">
+<collision>
+  <origin xyz="0 0 0" rpy="0 0 0"/>
+  <geometry>
+    <box size="0.1 0.1 0.1"/>
+  </geometry>
+</collision>
+<visual>
+  <origin xyz="0 0 0" rpy="0 0 0"/>
+  <geometry>
+    <mesh filename="package://rrbot_description/meshes/hokuyo.dae"/>
+  </geometry>
+</visual>
+<inertial>
+  <mass value="1e-5" />
+  <origin xyz="0 0 0" rpy="0 0 0"/>
+  <inertia ixx="1e-6" ixy="0" ixz="0" iyy="1e-6" iyz="0" izz="1e-6" />
+</inertial>
+</link-->
+<!--joint name="camera_joint" type="fixed">
+<axis xyz="0 1 0" />
+<origin xyz="${camera_link} 0 ${height3 - axel_offset*2}" rpy="0 0 0"/>
+<parent link="world"/>
+<child link="camera_link"/>
+</joint-->
+<!-- Camera -->
+<!--link name="camera_link">
+<collision>
+  <origin xyz="0 0 0" rpy="0 0 0"/>
+  <geometry>
+    <box size="${camera_link} ${camera_link} ${camera_link}"/>
+  </geometry>
+</collision>
+<visual>
+  <origin xyz="0 0 0" rpy="0 0 0"/>
+  <geometry>
+    <box size="${camera_link} ${camera_link} ${camera_link}"/>
+  </geometry>
+  <material name="red"/>
+</visual>
+<inertial>
+  <mass value="1e-5" />
+  <origin xyz="0 0 0" rpy="0 0 0"/>
+  <inertia ixx="1e-6" ixy="0" ixz="0" iyy="1e-6" iyz="0" izz="1e-6" />
+</inertial>
+</link-->
+<transmission name="tran1">
+  <type>transmission_interface/SimpleTransmission</type>
+  <joint name="joint1">
+    <hardwareInterface>EffortJointInterface</hardwareInterface>
+  </joint>
+  <actuator name="motor1">
+    <hardwareInterface>EffortJointInterface</hardwareInterface>
+    <mechanicalReduction>1</mechanicalReduction>
+  </actuator>
+</transmission>
+<transmission name="tran2">
+  <type>transmission_interface/SimpleTransmission</type>
+  <joint name="joint2">
+    <hardwareInterface>EffortJointInterface</hardwareInterface>
+  </joint>
+  <actuator name="motor2">
+    <hardwareInterface>EffortJointInterface</hardwareInterface>
+    <mechanicalReduction>1</mechanicalReduction>
+  </actuator>
+</transmission>
+<transmission name="tran3">
+  <type>transmission_interface/SimpleTransmission</type>
+  <joint name="joint3">
+    <hardwareInterface>EffortJointInterface</hardwareInterface>
+  </joint>
+  <actuator name="motor3">
+    <hardwareInterface>EffortJointInterface</hardwareInterface>
+    <mechanicalReduction>1</mechanicalReduction>
+  </actuator>
+</transmission>
+<transmission name="tran4">
+  <type>transmission_interface/SimpleTransmission</type>
+  <joint name="joint4">
+    <hardwareInterface>EffortJointInterface</hardwareInterface>
+  </joint>
+  <actuator name="motor4">
+    <hardwareInterface>EffortJointInterface</hardwareInterface>
+    <mechanicalReduction>1</mechanicalReduction>
+  </actuator>
+</transmission>
 </robot>

Commit message: Fix bugs

File: src/gazebo_ros_demos/rrbot_description/urdf/rrbot.xacro (robot description, xacro)
@@ -108,20 +108,20 @@
   <link name="link4">
     <collision>
-      <origin xyz="0.00 0 0.0" rpy="0 ${PI*0.5} 0"/>
-      <geometry>
-        <cylinder radius='${wheel_radius*1.4}' length="0.02"/>
-      </geometry>
-    </collision>
-    <visual>
-      <origin xyz="0.00 0 0.00" rpy="0 ${PI*0.5} 0"/>
-      <geometry>
-        <cylinder radius='${wheel_radius*1.4}' length="0.02"/>
+      <origin xyz="0.00 0 0.0" rpy="0 ${PI*0.0} 0"/>
+      <geometry>
+        <cylinder radius='${wheel_radius*1.5}' length="0.02"/>
+      </geometry>
+    </collision>
+    <visual>
+      <origin xyz="0.00 0 0.00" rpy="0 ${PI*0.0} 0"/>
+      <geometry>
+        <cylinder radius='${wheel_radius*1.5}' length="0.02"/>
       </geometry>
       <material name="red"/>
     </visual>
     <inertial>
-      <origin xyz="0.00 0 0.00" rpy="0 ${PI*0.5} 0"/>
+      <origin xyz="0.00 0 0.00" rpy="0 ${PI*0.0} 0"/>
       <mass value="${0.001*mass}"/>
-      <inertia	  ixx="1" ixy="0.0" ixz="0.0"	  iyy="1" iyz="0.0"	  izz="1"/>
+      <inertia	  ixx="0.1" ixy="0.0" ixz="0.0"	  iyy="0.1" iyz="0.0"	  izz="0.1"/>
     </inertial>
   </link>
@@ -129,33 +129,47 @@
     <parent link="link2"/>
     <child link="link4"/>
-    <origin xyz="${base_link_size_x*3/2} 0 0 " rpy="${PI*0.0} ${PI*0.0} ${PI*0.0}"/>
-    <axis xyz="1 0 0"/>
+    <origin xyz="${base_link_size_x*3/2} 0 0 " rpy="${PI*0.0} ${PI*0.5} ${PI*0.0}"/>
+    <axis xyz="0 0 1"/>
     <!--limit lower="${-PI}" upper="${PI}" effort="100" velocity="1"/-->
   </joint>
   <link name="link5">
-    <collision>
-      <origin xyz="0.00 0 0.0" rpy="0 ${PI*0.5} 0"/>
-      <geometry>
-        <cylinder radius='${wheel_radius*1.4}' length="0.02"/>
-      </geometry>
-    </collision>
-    <visual>
-      <origin xyz="0.00 0 0.00" rpy="0 ${PI*0.5} 0"/>
-      <geometry>
-        <cylinder radius='${wheel_radius*1.4}' length="0.02"/>
+    <inertial>
+      <origin xyz="0.00 0 0.00" rpy="0 ${PI*0.0} 0"/>
+      <mass value="${0.001*mass}"/>
+      <inertia	  ixx="0.1" ixy="0.0" ixz="0.0"	  iyy="0.1" iyz="0.0"	  izz="0.1"/>
+    </inertial>
+    <collision>
+      <origin xyz="0.00 0 0.0" rpy="0 ${PI*0.0} 0"/>
+      <geometry>
+        <cylinder radius='${wheel_radius*1.5}' length="0.02"/>
+      </geometry>
+      <surface>
+          <contact>
+            <ode/>
+          </contact>
+          <friction>
+            <ode/>
+          </friction>
+        </surface>
+    </collision>
+    <visual>
+      <origin xyz="0.00 0 0.00" rpy="0 ${PI*0.0} 0"/>
+      <geometry>
+        <cylinder radius='${wheel_radius*1.5}' length="0.02"/>
       </geometry>
       <material name="red"/>
     </visual>
-    <inertial>
-      <origin xyz="0.00 0 0.00" rpy="0 ${PI*0.5} 0"/>
-      <mass value="${0.001*mass}"/>
-      <inertia	  ixx="1" ixy="0.0" ixz="0.0"	  iyy="1" iyz="0.0"	  izz="1"/>
-    </inertial>
+    <gravity>1</gravity>
+      <velocity_decay>
+        <linear>0.000000</linear>
+        <angular>0.000000</angular>
+      </velocity_decay>
+      <self_collide>0</self_collide>
   </link>
   <joint name="joint4" type="continuous">
     <parent link="link3"/>
     <child link="link5"/>
-    <origin xyz="${-base_link_size_x*3/2} 0 0 " rpy="${PI*0.0} ${PI*0.0} ${PI*0.0}"/>
-    <axis xyz="1 0 0"/>
+    <origin xyz="${-base_link_size_x*3/2} 0 0 " rpy="${PI*0.0} ${PI*0.5} ${PI*0.0}"/>
+    <axis xyz="0 0 1"/>
   </joint>
   <!--joint name="hokuyo_joint" type="fixed">
