Commit message: Create 6 wheels

File: src/gazebo_ros_demos/rrbot_description/urdf/rrbot.xacro (robot description, xacro)
@@ -32,5 +32,5 @@
   <!-- Import Rviz colors -->
   <xacro:include filename="$(find rrbot_description)/urdf/materials.xacro" />
-  <link name="link1">
+  <link name="base_link">
     <visual>
       <origin xyz="0 0 0" rpy="0 0 0 "/>
@@ -53,11 +53,11 @@
   </link>
   <joint name="joint1" type="revolute">
-    <parent link="link1"/>
-    <child link="link2"/>
+    <parent link="base_link"/>
+    <child link="left_flipper"/>
     <origin xyz="0 0 0 " rpy="${PI*0.0} ${PI*0.0} ${PI*0.0}"/>
     <axis xyz="1 0 0"/>
     <limit lower="${-PI*0.5}" upper="${PI*0.5}" effort="100" velocity="1"/>
   </joint>
-  <link name="link2">
+  <link name="left_flipper">
     <collision>
       <origin xyz="0 0 0" rpy="0 0 0"/>
@@ -80,11 +80,11 @@
   </link>
   <joint name="joint2" type="revolute">
-    <parent link="link1"/>
-    <child link="link3"/>
+    <parent link="base_link"/>
+    <child link="right_flipper"/>
     <origin xyz="0 0 0" rpy="0 0 0"/>
     <axis xyz="1 0 0"/>
     <limit lower="${-PI*0.5}" upper="${PI*0.5}" effort="100" velocity="1"/>
   </joint>
-  <link name="link3">
+  <link name="right_flipper">
     <collision>
       <origin xyz="0 0 0" rpy="0 0 0"/>
@@ -106,5 +106,5 @@
     </inertial>
   </link>
-  <link name="link4">
+  <link name="right_front_wheel">
     <collision>
       <origin xyz="0.00 0 0.0" rpy="0 ${PI*0.0} 0"/>
@@ -127,11 +127,11 @@
   </link>
   <joint name="joint3" type="continuous">
-    <parent link="link2"/>
-    <child link="link4"/>
-    <origin xyz="${base_link_size_x*3/2} 0 0 " rpy="${PI*0.0} ${PI*0.5} ${PI*0.0}"/>
+    <parent link="left_flipper"/>
+    <child link="right_front_wheel"/>
+    <origin xyz="${base_link_size_x*1.25} 0 0 " rpy="${PI*0.0} ${PI*0.5} ${PI*0.0}"/>
     <axis xyz="0 0 1"/>
     <!--limit lower="${-PI}" upper="${PI}" effort="100" velocity="1"/-->
   </joint>
-  <link name="link5">
+  <link name="left_front_wheel">
     <inertial>
       <origin xyz="0.00 0 0.00" rpy="0 ${PI*0.0} 0"/>
@@ -168,63 +168,110 @@
   </link>
   <joint name="joint4" type="continuous">
-    <parent link="link3"/>
-    <child link="link5"/>
-    <origin xyz="${-base_link_size_x*3/2} 0 0 " rpy="${PI*0.0} ${PI*0.5} ${PI*0.0}"/>
-    <axis xyz="0 0 1"/>
-  </joint>
-  <!--joint name="hokuyo_joint" type="fixed">
-  <axis xyz="0 1 0" />
-  <origin xyz="0 0 ${height3 - axel_offset/2}" rpy="0 0 0"/>
-  <parent link="world"/>
-  <child link="hokuyo_link"/>
-</joint-->
-<!-- Hokuyo Laser -->
-<!--link name="hokuyo_link">
-<collision>
-  <origin xyz="0 0 0" rpy="0 0 0"/>
-  <geometry>
-    <box size="0.1 0.1 0.1"/>
-  </geometry>
-</collision>
-<visual>
-  <origin xyz="0 0 0" rpy="0 0 0"/>
-  <geometry>
-    <mesh filename="package://rrbot_description/meshes/hokuyo.dae"/>
-  </geometry>
-</visual>
-<inertial>
-  <mass value="1e-5" />
-  <origin xyz="0 0 0" rpy="0 0 0"/>
-  <inertia ixx="1e-6" ixy="0" ixz="0" iyy="1e-6" iyz="0" izz="1e-6" />
-</inertial>
-</link-->
-<!--joint name="camera_joint" type="fixed">
-<axis xyz="0 1 0" />
-<origin xyz="${camera_link} 0 ${height3 - axel_offset*2}" rpy="0 0 0"/>
-<parent link="world"/>
-<child link="camera_link"/>
-</joint-->
-<!-- Camera -->
-<!--link name="camera_link">
-<collision>
-  <origin xyz="0 0 0" rpy="0 0 0"/>
-  <geometry>
-    <box size="${camera_link} ${camera_link} ${camera_link}"/>
-  </geometry>
-</collision>
-<visual>
-  <origin xyz="0 0 0" rpy="0 0 0"/>
-  <geometry>
-    <box size="${camera_link} ${camera_link} ${camera_link}"/>
-  </geometry>
-  <material name="red"/>
-</visual>
-<inertial>
-  <mass value="1e-5" />
-  <origin xyz="0 0 0" rpy="0 0 0"/>
-  <inertia ixx="1e-6" ixy="0" ixz="0" iyy="1e-6" iyz="0" izz="1e-6" />
-</inertial>
-</link-->
-<transmission name="tran1">
+    <parent link="right_flipper"/>
+    <child link="left_front_wheel"/>
+    <origin xyz="${-base_link_size_x*1.25} 0 0 " rpy="${PI*0.0} ${PI*0.5} ${PI*0.0}"/>
+    <axis xyz="0 0 1"/>
+  </joint>
+  <link name="left_rear_wheel">
+    <inertial>
+      <origin xyz="0.00 0 0.00" rpy="0 ${PI*0.0} 0"/>
+      <mass value="${0.001*mass}"/>
+      <inertia	  ixx="0.1" ixy="0.0" ixz="0.0"	  iyy="0.1" iyz="0.0"	  izz="0.1"/>
+    </inertial>
+    <collision>
+      <origin xyz="0.00 0 0.0" rpy="0 ${PI*0.0} 0"/>
+      <geometry>
+        <cylinder radius='${wheel_radius*1.5}' length="0.02"/>
+      </geometry>
+    </collision>
+    <visual>
+      <origin xyz="0.00 0 0.00" rpy="0 ${PI*0.0} 0"/>
+      <geometry>
+        <cylinder radius='${wheel_radius*1.5}' length="0.02"/>
+      </geometry>
+    </visual>
+  </link>
+  <joint name="joint5" type="continuous">
+    <parent link="base_link"/>
+    <child link="left_rear_wheel"/>
+    <origin xyz="${-base_link_size_x*1.25} ${-base_link_size_y} 0 " rpy="${PI*0.0} ${PI*0.5} ${PI*0.0}"/>
+    <axis xyz="0 0 1"/>
+  </joint>
+  <link name="right_rear_wheel">
+    <inertial>
+      <origin xyz="0.00 0 0.00" rpy="0 ${PI*0.0} 0"/>
+      <mass value="${0.001*mass}"/>
+      <inertia	  ixx="0.1" ixy="0.0" ixz="0.0"	  iyy="0.1" iyz="0.0"	  izz="0.1"/>
+    </inertial>
+    <collision>
+      <origin xyz="0.00 0 0.0" rpy="0 ${PI*0.0} 0"/>
+      <geometry>
+        <cylinder radius='${wheel_radius*1.5}' length="0.02"/>
+      </geometry>
+    </collision>
+    <visual>
+      <origin xyz="0.00 0 0.00" rpy="0 ${PI*0.0} 0"/>
+      <geometry>
+        <cylinder radius='${wheel_radius*1.5}' length="0.02"/>
+      </geometry>
+    </visual>
+  </link>
+  <joint name="joint6" type="continuous">
+    <parent link="base_link"/>
+    <child link="right_rear_wheel"/>
+    <origin xyz="${base_link_size_x*1.25} ${-base_link_size_y} 0 " rpy="${PI*0.0} ${PI*0.5} ${PI*0.0}"/>
+    <axis xyz="0 0 1"/>
+  </joint>
+  <link name="left_flipper_wheel">
+    <inertial>
+      <origin xyz="0.00 0 0.00" rpy="0 ${PI*0.0} 0"/>
+      <mass value="${0.001*mass}"/>
+      <inertia	  ixx="0.1" ixy="0.0" ixz="0.0"	  iyy="0.1" iyz="0.0"	  izz="0.1"/>
+    </inertial>
+    <collision>
+      <origin xyz="0.00 0 0.0" rpy="0 ${PI*0.0} 0"/>
+      <geometry>
+        <cylinder radius='${wheel_radius*0.9}' length="0.02"/>
+      </geometry>
+    </collision>
+    <visual>
+      <origin xyz="0.00 0 0.00" rpy="0 ${PI*0.0} 0"/>
+      <geometry>
+        <cylinder radius='${wheel_radius*0.9}' length="0.02"/>
+      </geometry>
+    </visual>
+  </link>
+  <joint name="joint7" type="continuous">
+    <parent link="left_flipper"/>
+    <child link="left_flipper_wheel"/>
+    <origin xyz="-0.25 0.35 0 " rpy="${PI*0.0} ${PI*0.5} ${PI*0.0}"/>
+    <axis xyz="0 0 1"/>
+  </joint>
+  <link name="right_flipper_wheel">
+    <inertial>
+      <origin xyz="0.00 0 0.00" rpy="0 ${PI*0.0} 0"/>
+      <mass value="${0.001*mass}"/>
+      <inertia	  ixx="0.1" ixy="0.0" ixz="0.0"	  iyy="0.1" iyz="0.0"	  izz="0.1"/>
+    </inertial>
+    <collision>
+      <origin xyz="0.00 0 0.0" rpy="0 ${PI*0.0} 0"/>
+      <geometry>
+        <cylinder radius='${wheel_radius*0.9}' length="0.02"/>
+      </geometry>
+    </collision>
+    <visual>
+      <origin xyz="0.00 0 0.00" rpy="0 ${PI*0.0} 0"/>
+      <geometry>
+        <cylinder radius='${wheel_radius*0.9}' length="0.02"/>
+      </geometry>
+    </visual>
+  </link>
+  <joint name="joint8" type="continuous">
+    <parent link="right_flipper"/>
+    <child link="right_flipper_wheel"/>
+    <origin xyz="0.25 0.35 0 " rpy="${PI*0.0} ${PI*0.5} ${PI*0.0}"/>
+    <axis xyz="0 0 1"/>
+  </joint>
+  <transmission name="tran1">
   <type>transmission_interface/SimpleTransmission</type>
   <joint name="joint1">
@@ -266,3 +313,43 @@
   </actuator>
 </transmission>
+<transmission name="tran5">
+  <type>transmission_interface/SimpleTransmission</type>
+  <joint name="joint5">
+    <hardwareInterface>EffortJointInterface</hardwareInterface>
+  </joint>
+  <actuator name="motor5">
+    <hardwareInterface>EffortJointInterface</hardwareInterface>
+    <mechanicalReduction>1</mechanicalReduction>
+  </actuator>
+</transmission>
+<transmission name="tran6">
+  <type>transmission_interface/SimpleTransmission</type>
+  <joint name="joint6">
+    <hardwareInterface>EffortJointInterface</hardwareInterface>
+  </joint>
+  <actuator name="motor6">
+    <hardwareInterface>EffortJointInterface</hardwareInterface>
+    <mechanicalReduction>1</mechanicalReduction>
+  </actuator>
+</transmission>
+<transmission name="tran7">
+  <type>transmission_interface/SimpleTransmission</type>
+  <joint name="joint7">
+    <hardwareInterface>EffortJointInterface</hardwareInterface>
+  </joint>
+  <actuator name="motor7">
+    <hardwareInterface>EffortJointInterface</hardwareInterface>
+    <mechanicalReduction>1</mechanicalReduction>
+  </actuator>
+</transmission>
+<transmission name="tran8">
+  <type>transmission_interface/SimpleTransmission</type>
+  <joint name="joint8">
+    <hardwareInterface>EffortJointInterface</hardwareInterface>
+  </joint>
+  <actuator name="motor8">
+    <hardwareInterface>EffortJointInterface</hardwareInterface>
+    <mechanicalReduction>1</mechanicalReduction>
+  </actuator>
+</transmission>
 </robot>
