Commit message: Create self-collide

File: src/gazebo_ros_demos/rrbot_description/urdf/rrbot.xacro (robot description, xacro)
@@ -49,5 +49,6 @@
             <xacro:visual_macro mesh_name="${mesh_name}" x="${x}" y="${y}" z="${z}" roll="0" pitch="0" yaw="0"
                                 material="${material}" scale="${scale}"/>
-            <xacro:collision_macro mesh_name="${mesh_name}" x="${x}" y="${y}" z="${z}" roll="0" pitch="0" yaw="0" scale="${scale}"/>
+            <xacro:collision_macro mesh_name="${mesh_name}" x="${x}" y="${y}" z="${z}" roll="0" pitch="0" yaw="0"
+                                   scale="${scale}"/>
             <xacro:inertial_macro x="${x}" y="${y}" z="${z}"
                                   roll="0" pitch="0" yaw="0" mass="${mass}"
@@ -79,8 +80,8 @@
         <link name="${name_link}">
             <visual>
-              <origin xyz="0 0 0" rpy="0 0 0"/>
-              <geometry>
-                <cylinder radius='${radius}' length="${wheel_length}"/>
-              </geometry>
+                <origin xyz="0 0 0" rpy="0 0 0"/>
+                <geometry>
+                    <cylinder radius='${radius}' length="${wheel_length}"/>
+                </geometry>
             </visual>
             <collision>
@@ -113,7 +114,7 @@
     </xacro:macro>
     <xacro:link_macro name_link="base_link" x="0" y="0" z="0" mesh_name="Base.dae" mass="10" material="orange"
-                      scale="1" ixx="1" ixy="0.0" ixz="0.0" iyy="1" iyz="0.000" izz="1" />
+                      scale="1" ixx="1" ixy="0.0" ixz="0.0" iyy="1" iyz="0.000" izz="1"/>
     <xacro:link_macro name_link="right_flipper" x="0" y="0" z="0" mesh_name="Flipper.dae" mass="0.775" material="black"
-                      scale="1" ixx="1" ixy="0.0" ixz="0.0" iyy="1" iyz="0.000" izz="1" />
+                      scale="1" ixx="1" ixy="0.0" ixz="0.0" iyy="1" iyz="0.000" izz="1"/>
     <xacro:joint_macro joint_name="joint_right_flipper" type="revolute" parent="base_link" child="right_flipper"
                        x="2.2" y="1.86" z="-0.25" roll="0" pitch="0" yaw="0" axis="1 0 0"/>
@@ -135,18 +136,19 @@
                  radius="${small_wheel_radius}" wheel_length="0.2" mass="0.0001" parent="left_flipper"/>
     <xacro:link_macro name_link="cronstein" x="0" y="0" z="0" mesh_name="cronstain2.dae" mass="0.477" material="red"
-                      scale="1" ixx="1" ixy="0.0" ixz="0.0" iyy="1" iyz="0.000" izz="1"  />
+                      scale="1" ixx="1" ixy="0.0" ixz="0.0" iyy="1" iyz="0.000" izz="1"/>
     <xacro:joint_macro joint_name="joint_cronstein" type="revolute" parent="base_link" child="cronstein"
                        x="0" y="-1.75" z="0.6" roll="0" pitch="${PI*0.5}" yaw="${PI*0.5}" axis="1 0 0"/>
-    <!--x="0.5" y="-1.05" z="1.1" roll="0" pitch="${PI*0.5}" yaw="${PI*0.5}" axis="0 0 1"/>-->
-    <xacro:link_macro name_link="first_part" x="0" y="0" z="0" mesh_name="first_part_of_arm.dae" mass="2.231" material="red"
-                      scale="0.01" ixx="1" ixy="0.0" ixz="0.0" iyy="1" iyz="0.000" izz="1"  />
+    <xacro:link_macro name_link="first_part" x="0" y="0" z="0" mesh_name="first_part_of_arm.dae" mass="2.231"
+                      material="red"
+                      scale="0.01" ixx="1" ixy="0.0" ixz="0.0" iyy="1" iyz="0.000" izz="1"/>
     <xacro:joint_macro joint_name="joint_first_part" type="revolute" parent="cronstein" child="first_part"
                        x="-0.54" y="0.25" z="0.7" roll="${PI}" pitch="${PI}" yaw="${PI*0.5}" axis="1 0 0"/>
-    <xacro:link_macro name_link="second_part" x="0" y="0" z="0" mesh_name="second_part_of_arm.dae" mass="2.231" material="red"
-                      scale="0.01" ixx="1" ixy="0.0" ixz="0.0" iyy="1" iyz="0.000" izz="1"  />
+    <xacro:link_macro name_link="second_part" x="0" y="0" z="0" mesh_name="second_part_of_arm.dae" mass="1.407"
+                      material="red"
+                      scale="0.01" ixx="1" ixy="0.0" ixz="0.0" iyy="1" iyz="0.000" izz="1"/>
     <xacro:joint_macro joint_name="joint_second_part" type="revolute" parent="first_part" child="second_part"
                        x="-1.5" y="0" z="3" roll="0" pitch="0" yaw="${PI}" axis="1 0 0"/>
-    <xacro:link_macro name_link="head" x="0" y="0" z="0" mesh_name="head.dae" mass="2.231" material="red"
-                      scale="0.01" ixx="1" ixy="0.0" ixz="0.0" iyy="1" iyz="0.000" izz="1"  />
+    <xacro:link_macro name_link="head" x="0" y="0" z="0" mesh_name="head.dae" mass="4.738" material="red"
+                      scale="0.01" ixx="1" ixy="0.0" ixz="0.0" iyy="1" iyz="0.000" izz="1"/>
     <xacro:joint_macro joint_name="joint_head" type="revolute" parent="second_part" child="head"
                        x="0.5" y="0" z="-4.2" roll="${PI}" pitch="${PI*0}" yaw="${PI}" axis="1 0 0"/>

Commit message: Update code

File: src/gazebo_ros_demos/rrbot_description/urdf/rrbot.xacro (robot description, xacro)
@@ -79,10 +79,10 @@
                  params="name_link x y z roll pitch yaw radius wheel_length mass parent">
         <link name="${name_link}">
-            <visual>
-                <origin xyz="0 0 0" rpy="0 0 0"/>
-                <geometry>
-                    <cylinder radius='${radius}' length="${wheel_length}"/>
-                </geometry>
-            </visual>
+            <!--<visual>-->
+                <!--<origin xyz="0 0 0" rpy="0 0 0"/>-->
+                <!--<geometry>-->
+                    <!--<cylinder radius='${radius}' length="${wheel_length}"/>-->
+                <!--</geometry>-->
+            <!--</visual>-->
             <collision>
                 <origin xyz="0 0 0" rpy="0 0 0"/>

Commit message: Big update: Rebuild 3d model

File: src/gazebo_ros_demos/rrbot_description/urdf/rrbot.xacro (robot description, xacro)
@@ -1,4 +1,4 @@
 <?xml version="1.0" encoding="UTF-8"?>
-<!-- Revolute-Revolute Manipulator -->
+<!-- continuous-continuous Manipulator -->
 <robot name="rrbot" xmlns:xacro="http://www.ros.org/wiki/xacro">
     <!-- Constants for robot dimensions -->
@@ -63,5 +63,5 @@
             <origin xyz="${x} ${y} ${z}" rpy="${roll} ${pitch} ${yaw}"/>
             <axis xyz="${axis}"/>
-            <limit lower="${-2*PI}" upper="${2*PI}" effort="100" velocity="100"/>
+            <limit lower="${-2*PI}" upper="${2*PI}" effort="1000" velocity="1000"/>
         </joint>
         <transmission name="tran_${joint_name}">
@@ -79,10 +79,10 @@
                  params="name_link x y z roll pitch yaw radius wheel_length mass parent">
         <link name="${name_link}">
-            <!--<visual>-->
-                <!--<origin xyz="0 0 0" rpy="0 0 0"/>-->
-                <!--<geometry>-->
-                    <!--<cylinder radius='${radius}' length="${wheel_length}"/>-->
-                <!--</geometry>-->
-            <!--</visual>-->
+            <!-- <visual>
+                <origin xyz="0 0 0" rpy="0 0 0"/>
+                <geometry>
+                    <cylinder radius='${radius}' length="${wheel_length}"/>
+                 </geometry>
+            </visual> -->
             <collision>
                 <origin xyz="0 0 0" rpy="0 0 0"/>
@@ -115,12 +115,12 @@
     <xacro:link_macro name_link="base_link" x="0" y="0" z="0" mesh_name="Base.dae" mass="10" material="orange"
                       scale="1" ixx="1" ixy="0.0" ixz="0.0" iyy="1" iyz="0.000" izz="1"/>
-    <xacro:link_macro name_link="right_flipper" x="0" y="0" z="0" mesh_name="Flipper.dae" mass="0.775" material="black"
+    <xacro:link_macro name_link="right_flipper" x="0" y="0" z="0" mesh_name="RightFlipper.dae" mass="0.775" material="grey"
                       scale="1" ixx="1" ixy="0.0" ixz="0.0" iyy="1" iyz="0.000" izz="1"/>
-    <xacro:joint_macro joint_name="joint_right_flipper" type="revolute" parent="base_link" child="right_flipper"
-                       x="2.2" y="1.86" z="-0.25" roll="0" pitch="0" yaw="0" axis="1 0 0"/>
-    <xacro:link_macro name_link="left_flipper" x="0" y="0" z="0" mesh_name="Flipper.dae" mass="0.775" material="black"
+    <xacro:joint_macro joint_name="joint_right_flipper" type="continuous" parent="base_link" child="right_flipper"
+                       x="2.2" y="1.86" z="-0.25" roll="${-PI*0.5}" pitch="0" yaw="0" axis="1 0 0" />
+    <xacro:link_macro name_link="left_flipper" x="0" y="0" z="0" mesh_name="LeftFlipper.dae" mass="0.775" material="grey"
                       scale="1" ixx="1" ixy="0.0" ixz="0.0" iyy="1" iyz="0.000" izz="1"/>
-    <xacro:joint_macro joint_name="joint_left_flipper" type="revolute" parent="base_link" child="left_flipper"
-                       x="-2.2" y="1.86" z="-0.25" roll="0" pitch="${PI}" yaw="0" axis="1 0 0"/>
+    <xacro:joint_macro joint_name="joint_left_flipper" type="continuous" parent="base_link" child="left_flipper"
+                       x="-2.2" y="1.86" z="-0.25" roll="${-PI*0.5}" pitch="0" yaw="0" axis="1 0 0"/>
     <xacro:wheel name_link="right_front_base_link_wheel" x="4" y="1.86" z="-0.25" roll="0" pitch="${PI*0.5}" yaw="${PI}"
                  radius="${big_wheel_radius}" wheel_length="0.2" mass="0.0001" parent="base_link"/>
@@ -131,25 +131,26 @@
     <xacro:wheel name_link="left_rear_base_link_wheel" x="-4" y="-1.86" z="-0.25" roll="0" pitch="${PI*0.5}" yaw="${PI}"
                  radius="${big_wheel_radius}" wheel_length="0.2" mass="0.0001" parent="base_link"/>
-    <xacro:wheel name_link="right_flipper_wheel" x="0.3" y="3.4" z="0" roll="0" pitch="${PI*0.5}" yaw="${PI}"
+<!-- y=3.4 x=0.3-->
+    <xacro:wheel name_link="right_flipper_wheel" x="0.5" y="0" z="3.4" roll="0" pitch="${PI*0.5}" yaw="${PI}"
                  radius="${small_wheel_radius}" wheel_length="0.2" mass="0.0001" parent="right_flipper"/>
-    <xacro:wheel name_link="left_flipper_wheel" x="0.3" y="3.4" z="0" roll="0" pitch="${PI*0.5}" yaw="${PI}"
+    <xacro:wheel name_link="left_flipper_wheel" x="-0.5" y="0" z="3.4" roll="0" pitch="${PI*0.5}" yaw="${PI}"
                  radius="${small_wheel_radius}" wheel_length="0.2" mass="0.0001" parent="left_flipper"/>
-    <xacro:link_macro name_link="cronstein" x="0" y="0" z="0" mesh_name="cronstain2.dae" mass="0.477" material="red"
+    <xacro:link_macro name_link="cronstein" x="0" y="0" z="0" mesh_name="cronstain3.dae" mass="0.477" material="red"
                       scale="1" ixx="1" ixy="0.0" ixz="0.0" iyy="1" iyz="0.000" izz="1"/>
-    <xacro:joint_macro joint_name="joint_cronstein" type="revolute" parent="base_link" child="cronstein"
-                       x="0" y="-1.75" z="0.6" roll="0" pitch="${PI*0.5}" yaw="${PI*0.5}" axis="1 0 0"/>
+    <xacro:joint_macro joint_name="joint_cronstein" type="continuous" parent="base_link" child="cronstein"
+      x="0" y="-1.75" z="0.37" roll="0" pitch="${PI*0.0}" yaw="${PI*0.0}" axis="0 0 1"/>
     <xacro:link_macro name_link="first_part" x="0" y="0" z="0" mesh_name="first_part_of_arm.dae" mass="2.231"
                       material="red"
                       scale="0.01" ixx="1" ixy="0.0" ixz="0.0" iyy="1" iyz="0.000" izz="1"/>
-    <xacro:joint_macro joint_name="joint_first_part" type="revolute" parent="cronstein" child="first_part"
-                       x="-0.54" y="0.25" z="0.7" roll="${PI}" pitch="${PI}" yaw="${PI*0.5}" axis="1 0 0"/>
+    <xacro:joint_macro joint_name="joint_first_part" type="continuous" parent="cronstein" child="first_part"
+                       x="0.3" y="0.7" z="0.5" roll="${PI*0.5}" pitch="${PI}" yaw="${PI}" axis="1 0 0"/>
     <xacro:link_macro name_link="second_part" x="0" y="0" z="0" mesh_name="second_part_of_arm.dae" mass="1.407"
                       material="red"
                       scale="0.01" ixx="1" ixy="0.0" ixz="0.0" iyy="1" iyz="0.000" izz="1"/>
-    <xacro:joint_macro joint_name="joint_second_part" type="revolute" parent="first_part" child="second_part"
-                       x="-1.5" y="0" z="3" roll="0" pitch="0" yaw="${PI}" axis="1 0 0"/>
+    <xacro:joint_macro joint_name="joint_second_part" type="continuous" parent="first_part" child="second_part"
+                       x="-0.7" y="0" z="3" roll="0" pitch="0" yaw="0" axis="1 0 0"/>
     <xacro:link_macro name_link="head" x="0" y="0" z="0" mesh_name="head.dae" mass="4.738" material="red"
                       scale="0.01" ixx="1" ixy="0.0" ixz="0.0" iyy="1" iyz="0.000" izz="1"/>
-    <xacro:joint_macro joint_name="joint_head" type="revolute" parent="second_part" child="head"
-                       x="0.5" y="0" z="-4.2" roll="${PI}" pitch="${PI*0}" yaw="${PI}" axis="1 0 0"/>
+    <xacro:joint_macro joint_name="joint_head" type="continuous" parent="second_part" child="head"
+                       x="0.2" y="0" z="-4.2" roll="${PI}" pitch="${PI*0}" yaw="0" axis="1 0 0"/>
 </robot>

Commit message: Add cube

File: src/gazebo_ros_demos/rrbot_description/urdf/rrbot.xacro (robot description, xacro)
@@ -13,7 +13,8 @@
                     value="${2*wheel_radius-ground_clearance}"/>   <!-- old 0.102 is double radius without ground_clearance 0.07683 -->
     <xacro:property name="big_wheel_radius" value="0.8"/>   <!--was 0.09-->
-    <xacro:property name="small_wheel_radius" value="0.5"/>   <!--was 0.09-->
+    <xacro:property name="small_wheel_radius" value="${big_wheel_radius*0.7}"/>   <!--was 0.09-->
     <xacro:property name="ground_clearance" value="0.02517"/>   <!--old 0.05 0.02517-->
     <xacro:property name="wheel_length" value="0.29"/>
+    <xacro:property name="wheel_mass" value="0.1"/>
     <xacro:include filename="$(find rrbot_description)/urdf/rrbot.gazebo"/>
     <xacro:include filename="$(find rrbot_description)/urdf/materials.xacro"/>
@@ -79,10 +80,10 @@
                  params="name_link x y z roll pitch yaw radius wheel_length mass parent">
         <link name="${name_link}">
-            <!-- <visual>
+            <visual>
                 <origin xyz="0 0 0" rpy="0 0 0"/>
                 <geometry>
                     <cylinder radius='${radius}' length="${wheel_length}"/>
                  </geometry>
-            </visual> -->
+            </visual>
             <collision>
                 <origin xyz="0 0 0" rpy="0 0 0"/>
@@ -123,21 +124,21 @@
     <xacro:joint_macro joint_name="joint_left_flipper" type="continuous" parent="base_link" child="left_flipper"
                        x="-2.2" y="1.86" z="-0.25" roll="${-PI*0.5}" pitch="0" yaw="0" axis="1 0 0"/>
-    <xacro:wheel name_link="right_front_base_link_wheel" x="4" y="1.86" z="-0.25" roll="0" pitch="${PI*0.5}" yaw="${PI}"
-                 radius="${big_wheel_radius}" wheel_length="0.2" mass="0.0001" parent="base_link"/>
-    <xacro:wheel name_link="left_front_base_link_wheel" x="-4" y="1.86" z="-0.25" roll="0" pitch="${PI*0.5}" yaw="${PI}"
-                 radius="${big_wheel_radius}" wheel_length="0.2" mass="0.0001" parent="base_link"/>
-    <xacro:wheel name_link="right_rear_base_link_wheel" x="4" y="-1.86" z="-0.25" roll="0" pitch="${PI*0.5}" yaw="${PI}"
-                 radius="${big_wheel_radius}" wheel_length="0.2" mass="0.0001" parent="base_link"/>
-    <xacro:wheel name_link="left_rear_base_link_wheel" x="-4" y="-1.86" z="-0.25" roll="0" pitch="${PI*0.5}" yaw="${PI}"
-                 radius="${big_wheel_radius}" wheel_length="0.2" mass="0.0001" parent="base_link"/>
+    <xacro:wheel name_link="right_front_base_link_wheel" x="2.75" y="1.86" z="-0.25" roll="0" pitch="${PI*0.5}" yaw="${PI}"
+                 radius="${big_wheel_radius}" wheel_length="0.2" mass="${wheel_mass}" parent="base_link"/>
+    <xacro:wheel name_link="left_front_base_link_wheel" x="-2.75" y="1.86" z="-0.25" roll="0" pitch="${PI*0.5}" yaw="${PI}"
+                 radius="${big_wheel_radius}" wheel_length="0.2" mass="${wheel_mass}" parent="base_link"/>
+    <xacro:wheel name_link="right_rear_base_link_wheel" x="2.75" y="-1.86" z="-0.25" roll="0" pitch="${PI*0.5}" yaw="${PI}"
+                 radius="${big_wheel_radius}" wheel_length="0.2" mass="${wheel_mass}" parent="base_link"/>
+    <xacro:wheel name_link="left_rear_base_link_wheel" x="-2.75" y="-1.86" z="-0.25" roll="0" pitch="${PI*0.5}" yaw="${PI}"
+                 radius="${big_wheel_radius}" wheel_length="0.2" mass="${wheel_mass}" parent="base_link"/>
 <!-- y=3.4 x=0.3-->
     <xacro:wheel name_link="right_flipper_wheel" x="0.5" y="0" z="3.4" roll="0" pitch="${PI*0.5}" yaw="${PI}"
-                 radius="${small_wheel_radius}" wheel_length="0.2" mass="0.0001" parent="right_flipper"/>
+                 radius="${small_wheel_radius}" wheel_length="0.2" mass="${wheel_mass}" parent="right_flipper"/>
     <xacro:wheel name_link="left_flipper_wheel" x="-0.5" y="0" z="3.4" roll="0" pitch="${PI*0.5}" yaw="${PI}"
-                 radius="${small_wheel_radius}" wheel_length="0.2" mass="0.0001" parent="left_flipper"/>
-    <xacro:link_macro name_link="cronstein" x="0" y="0" z="0" mesh_name="cronstain3.dae" mass="0.477" material="red"
+                 radius="${small_wheel_radius}" wheel_length="0.2" mass="${wheel_mass}" parent="left_flipper"/>
+    <!-- <xacro:link_macro name_link="cronstein" x="0" y="0" z="0" mesh_name="cronstain3.dae" mass="0.477" material="red"
                       scale="1" ixx="1" ixy="0.0" ixz="0.0" iyy="1" iyz="0.000" izz="1"/>
     <xacro:joint_macro joint_name="joint_cronstein" type="continuous" parent="base_link" child="cronstein"
-      x="0" y="-1.75" z="0.37" roll="0" pitch="${PI*0.0}" yaw="${PI*0.0}" axis="0 0 1"/>
+      x="0" y="-1.75" z="0.4" roll="0" pitch="${PI*0.0}" yaw="${PI*0.0}" axis="0 0 1"/>
     <xacro:link_macro name_link="first_part" x="0" y="0" z="0" mesh_name="first_part_of_arm.dae" mass="2.231"
                       material="red"
@@ -153,4 +154,4 @@
                       scale="0.01" ixx="1" ixy="0.0" ixz="0.0" iyy="1" iyz="0.000" izz="1"/>
     <xacro:joint_macro joint_name="joint_head" type="continuous" parent="second_part" child="head"
-                       x="0.2" y="0" z="-4.2" roll="${PI}" pitch="${PI*0}" yaw="0" axis="1 0 0"/>
+                       x="0.2" y="0" z="-4.2" roll="${PI}" pitch="${PI*0}" yaw="0" axis="1 0 0"/> -->
 </robot>

Commit message: Add XBox controller

File: src/gazebo_ros_demos/rrbot_description/urdf/rrbot.xacro (robot description, xacro)
@@ -33,5 +33,5 @@
             <origin xyz="${x} ${y} ${z}" rpy="${roll} ${pitch} ${yaw}"/>
             <mass value="${mass}"/>
-            <inertia ixx="${ixx}" ixy="${ixy}" ixz="${ixz}" iyy="${iyy}" iyz="${iyz}" izz="${izz}"/>
+            <inertia ixx="${mass}" ixy="0" ixz="0" iyy="${mass}" iyz="0" izz="${mass}"/>
         </inertial>
     </xacro:macro>
